File: IR_Tx.sch (KiCad schematic (older format))
At the start: 14 parts, among them P10 MOD, Q2 NPN, SW1 SW_STFU, U6 NE555

Commit message: WiP, added IR Tx parts on PCB.
Parts:
- BT1: footprint (none) -> CR2032
- C10, C9: footprint (none) -> cnp_3mm_disc
- C6: footprint (none) -> CP_5x11mm
- D62, D64: footprint (none) -> led_5mm_clear
- P10: footprint (none) -> pin_strip_2
- Q2: footprint (none) -> to92_2N5401
- R41, R6, R7: footprint (none) -> rc03_vert
- R5: footprint (none) -> pin_strip_3x2
- U6: footprint (none) -> DIP-8__300_ELL
Changed lines of the file:
@@
-EESchema Schematic File Version 2  date 7/18/2012 6:00:20 PM
+EESchema Schematic File Version 2  date Wednesday 18 July 2012 10:05:39 PM IST
 LIBS:stfu
 LIBS:power
@@
 F 0 "P10" V 5150 3250 40  0000 C CNN
 F 1 "MOD" V 5250 3250 40  0000 C CNN
+F 2 "pin_strip_2" H 5200 3250 60  0001 C CNN
 	1    5200 3250
 	-1   0    0    -1
@@
 F 0 "Q2" H 7550 3550 60  0000 R CNN
 F 1 "NPN" H 7550 3850 60  0000 R CNN
+F 2 "to92_2N5401" H 7550 3700 60  0001 C CNN
 	1    7550 3700
 	1    0    0    -1
@@
 F 0 "D62" V 7750 2800 50  0000 C CNN
 F 1 "LED" H 7500 2650 50  0000 C CNN
+F 2 "led_5mm_clear" H 7650 2700 60  0001 C CNN
 	1    7650 2700
 	0    1    1    0
@@
 F 0 "D64" V 7750 3300 50  0000 C CNN
 F 1 "LED" H 7500 3150 50  0000 C CNN
+F 2 "led_5mm_clear" H 7650 3200 60  0001 C CNN
 	1    7650 3200
 	0    1    1    0
@@
 F 0 "C9" H 4850 4500 50  0000 L CNN
 F 1 "1n" H 4850 4300 50  0000 L CNN
+F 2 "cnp_3mm_disc" H 4800 4400 60  0001 C CNN
 	1    4800 4400
 	1    0    0    -1
@@
 F 0 "C10" H 5200 4500 50  0000 L CNN
 F 1 "47n" H 5200 4300 50  0000 L CNN
+F 2 "cnp_3mm_disc" H 5150 4400 60  0001 C CNN
 	1    5150 4400
 	1    0    0    -1
@@
 F 0 "C6" H 4150 3850 50  0000 L CNN
 F 1 "10u" H 4150 3650 50  0000 L CNN
+F 2 "CP_5x11mm" H 4100 3750 60  0001 C CNN
 	1    4100 3750
 	1    0    0    -1
@@
 F 0 "R5" H 4900 2550 50  0000 C CNN
 F 1 "20k" V 4700 2650 50  0000 C CNN
+F 2 "pin_strip_3x2" H 4800 2650 60  0001 C CNN
 	1    4800 2650
 	1    0    0    -1
@@
 F 0 "R7" H 4900 3950 50  0000 C CNN
 F 1 "1k" V 4800 3850 50  0000 C CNN
+F 2 "rc03_vert" H 4800 3850 60  0001 C CNN
 	1    4800 3850
 	1    0    0    -1
@@
 F 0 "R6" H 4900 3350 50  0000 C CNN
 F 1 "10k" V 4800 3250 50  0000 C CNN
+F 2 "rc03_vert" H 4800 3250 60  0001 C CNN
 	1    4800 3250
 	1    0    0    -1
@@
 F 0 "R41" V 7080 3700 50  0000 C CNN
 F 1 "120E" V 7000 3700 50  0000 C CNN
+F 2 "rc03_vert" H 7000 3700 60  0001 C CNN
 	1    7000 3700
 	0    -1   -1   0
@@
 F 0 "BT1" H 3750 4000 50  0000 C CNN
 F 1 "BATT_Li" H 3750 3610 50  0000 C CNN
+F 2 "CR2032" H 3750 3800 60  0001 C CNN
 	1    3750 3800
 	0    1    1    0
@@
 F 0 "U6" H 6525 4250 60  0000 C CNN
 F 1 "NE555" H 6600 4150 60  0000 C CNN
+F 2 "DIP-8__300_ELL" H 6150 3800 60  0001 C CNN
 	1    6150 3800
 	1    0    0    -1

Commit message: WiP : STFU Ir Transmitter complete. BoM updated.
Parts:
- added R42: 47E, rc03_vert, symbol R
- added R43: 220E, rc03_vert, symbol R
- BT1: footprint CR2032 -> CR2032x2
- C6: value 10u -> 100n
- D64: value LED -> IR_LED
- SW1: footprint SW_PB_V -> SW-PB
Connections:
- wire segments 38 -> 42
Other:
- moved on the sheet: D62
Changed lines of the file:
@@
-EESchema Schematic File Version 2  date Wednesday 18 July 2012 10:05:39 PM IST
+EESchema Schematic File Version 2  date 7/19/2012 1:50:01 PM
 LIBS:stfu
 LIBS:power
@@
 Sheet 2 3
 Title ""
-Date "18 jul 2012"
+Date "19 jul 2012"
 Rev ""
 Comp ""
@@
 Comment4 ""
 $EndDescr
+Connection ~ 7650 3450
+Wire Wire Line
+	7650 3450 8000 3450
+Wire Wire Line
+	8000 3450 8000 3400
+Wire Wire Line
+	8000 3000 8000 2900
+Wire Wire Line
+	5600 2050 5600 3150
+Wire Wire Line
+	5550 3350 5600 3350
+Wire Wire Line
+	5600 3350 5600 3500
+Wire Wire Line
+	5600 3500 5650 3500
+Connection ~ 4100 4800
+Wire Wire Line
+	4100 3950 4100 4800
+Connection ~ 6150 4800
+Wire Wire Line
+	7650 4800 3750 4800
+Wire Wire Line
+	7650 4800 7650 3900
+Wire Wire Line
+	7650 3400 7650 3500
+Connection ~ 6150 2250
+Wire Wire Line
+	7650 2250 7650 2400
+Connection ~ 4800 3550
+Wire Wire Line
+	4800 3550 5000 3550
+Wire Wire Line
+	5000 3550 5000 3650
+Wire Wire Line
+	5000 3650 5650 3650
+Wire Wire Line
+	5000 3800 5000 4150
+Wire Wire Line
+	5000 3800 5650 3800
+Connection ~ 4800 2250
+Wire Wire Line
+	4800 3000 4800 2900
+Wire Wire Line
+	4800 4100 4800 4200
+Wire Wire Line
+	5150 4200 5150 4100
+Wire Wire Line
+	5150 4100 5650 4100
+Wire Wire Line
+	3750 4800 3750 4000
+Wire Wire Line
+	3750 3550 3750 3450
+Wire Wire Line
+	5150 4600 5150 4800
+Connection ~ 5150 4800
+Wire Wire Line
+	4800 3600 4800 3500
+Wire Wire Line
+	4800 2250 4800 2400
+Wire Wire Line
+	3750 2850 3750 2250
+Wire Wire Line
+	4950 2650 5050 2650
+Wire Wire Line
+	5050 2650 5050 2250
+Connection ~ 5050 2250
+Wire Wire Line
+	5000 3950 5650 3950
+Wire Wire Line
+	5000 4150 4800 4150
+Connection ~ 4800 4150
+Connection ~ 5000 3950
+Wire Wire Line
+	6650 3700 6750 3700
+Wire Wire Line
+	7650 2900 7650 3000
+Wire Wire Line
+	7350 3700 7250 3700
+Wire Wire Line
+	4100 3550 4100 2250
+Connection ~ 4100 2250
+Wire Wire Line
+	4800 4600 4800 4800
+Connection ~ 4800 4800
+Wire Wire Line
+	5600 3150 5550 3150
+Connection ~ 5600 2250
+Wire Wire Line
+	6150 3200 6150 2150
+Wire Wire Line
+	6150 4400 6150 5000
+Wire Wire Line
+	6500 4700 6500 4800
+Connection ~ 6500 4800
+Wire Wire Line
+	8000 2400 8000 2250
+Wire Wire Line
+	8000 2250 3750 2250
+Connection ~ 7650 2250
+$Comp
+L R R43
+U 1 1 5007B1DC
+P 8000 2650
+F 0 "R43" V 8080 2650 50  0000 C CNN
+F 1 "220E" V 8000 2650 50  0000 C CNN
+F 2 "rc03_vert" H 8000 2650 60  0001 C CNN
+	1    8000 2650
+	-1   0    0    1
+$EndComp
+$Comp
+L R R42
+U 1 1 5007B1C5
+P 7650 2650
+F 0 "R42" V 7730 2650 50  0000 C CNN
+F 1 "47E" V 7650 2650 50  0000 C CNN
+F 2 "rc03_vert" H 7650 2650 60  0001 C CNN
+	1    7650 2650
+	-1   0    0    1
+$EndComp
 Text Label 5600 3350 0    40   ~ 0
 RST
@@
 Text Label 4100 2250 0    60   ~ 0
 +6V
-Connection ~ 6500 4800
-Wire Wire Line
-	6500 4700 6500 4800
-Wire Wire Line
-	6150 5000 6150 4400
-Wire Wire Line
-	6150 2150 6150 3200
-Connection ~ 5600 2250
-Wire Wire Line
-	5550 3150 5600 3150
-Connection ~ 4800 4800
-Wire Wire Line
-	4800 4600 4800 4800
-Connection ~ 4100 2250
-Wire Wire Line
-	4100 3550 4100 2250
-Wire Wire Line
-	7350 3700 7250 3700
-Wire Wire Line
-	7650 2900 7650 3000
-Wire Wire Line
-	6650 3700 6750 3700
-Connection ~ 5000 3950
-Connection ~ 4800 4150
-Wire Wire Line
-	4800 4150 5000 4150
-Wire Wire Line
-	5000 3950 5650 3950
-Connection ~ 5050 2250
-Wire Wire Line
-	5050 2250 5050 2650
-Wire Wire Line
-	5050 2650 4950 2650
-Wire Wire Line
-	3750 2850 3750 2250
-Wire Wire Line
-	4800 2250 4800 2400
-Wire Wire Line
-	4800 3500 4800 3600
-Connection ~ 5150 4800
-Wire Wire Line
-	5150 4600 5150 4800
-Wire Wire Line
-	3750 3550 3750 3450
-Wire Wire Line
-	3750 4000 3750 4800
-Wire Wire Line
-	5650 4100 5150 4100
-Wire Wire Line
-	5150 4100 5150 4200
-Wire Wire Line
-	4800 4200 4800 4100
-Wire Wire Line
-	4800 3000 4800 2900
-Connection ~ 4800 2250
-Wire Wire Line
-	5650 3800 5000 3800
-Wire Wire Line
-	5000 3800 5000 4150
-Wire Wire Line
-	5650 3650 5000 3650
-Wire Wire Line
-	5000 3650 5000 3550
-Wire Wire Line
-	5000 3550 4800 3550
-Connection ~ 4800 3550
-Wire Wire Line
-	3750 2250 7650 2250
-Wire Wire Line
-	7650 2250 7650 2500
-Connection ~ 6150 2250
-Wire Wire Line
-	7650 3400 7650 3500
-Wire Wire Line
-	7650 3900 7650 4800
-Wire Wire Line
-	7650 4800 3750 4800
-Connection ~ 6150 4800
-Wire Wire Line
-	4100 3950 4100 4800
-Connection ~ 4100 4800
-Wire Wire Line
-	5650 3500 5600 3500
-Wire Wire Line
-	5600 3500 5600 3350
-Wire Wire Line
-	5600 3350 5550 3350
-Wire Wire Line
-	5600 3150 5600 2050
 $Comp
 L PWR_FLAG #FLG012
@@
 L LED D62
 U 1 1 5006A7EE
-P 7650 2700
-F 0 "D62" V 7750 2800 50  0000 C CNN
-F 1 "LED" H 7500 2650 50  0000 C CNN
-F 2 "led_5mm_clear" H 7650 2700 60  0001 C CNN
-	1    7650 2700
+P 8000 3200
+F 0 "D62" V 8100 3300 50  0000 C CNN
+F 1 "LED" H 7850 3150 50  0000 C CNN
+F 2 "led_5mm_clear" H 8000 3200 60  0001 C CNN
+	1    8000 3200
 	0    1    1    0
 $EndComp
@@
 P 7650 3200
 F 0 "D64" V 7750 3300 50  0000 C CNN
-F 1 "LED" H 7500 3150 50  0000 C CNN
+F 1 "IR_LED" H 7500 3150 50  0000 C CNN
 F 2 "led_5mm_clear" H 7650 3200 60  0001 C CNN
 	1    7650 3200
@@
 F 0 "SW1" H 3900 3260 50  0000 C CNN
 F 1 "SW_STFU" H 3750 3070 50  0000 C CNN
-F 2 "SW_PB_V" H 3800 3160 60  0001 C CNN
+F 2 "SW-PB" H 3800 3160 60  0001 C CNN
 F 3 "http://industrial.panasonic.com/www-data/pdf/ATK0000/ATK0000CE32.pdf" H 3900 3260 60  0001 C CNN
 F 4 "P10884S-ND" H 4000 3360 60  0001 C CNN "DigiKey"
@@
 P 4100 3750
 F 0 "C6" H 4150 3850 50  0000 L CNN
-F 1 "10u" H 4150 3650 50  0000 L CNN
+F 1 "100n" H 4150 3650 50  0000 L CNN
 F 2 "CP_5x11mm" H 4100 3750 60  0001 C CNN
 	1    4100 3750
@@
 U 1 1 5006A59F
 P 3750 3800
-F 0 "BT1" H 3750 4000 50  0000 C CNN
-F 1 "BATT_Li" H 3750 3610 50  0000 C CNN
-F 2 "CR2032" H 3750 3800 60  0001 C CNN
+F 0 "BT1" V 3650 3650 50  0000 C CNN
+F 1 "BATT_Li" V 3800 3600 50  0000 C CNN
+F 2 "CR2032x2" H 3750 3800 60  0001 C CNN
 	1    3750 3800
 	0    1    1    0

Commit message: WiP - track cleanup and optimization, Legend clean up etc.
Parts:
- C10, C9: footprint cnp_3mm_disc -> c_0805
- C6: footprint CP_5x11mm -> c_0805
- R41, R43: footprint rc03_vert -> r_0805
- R42: footprint rc03_vert -> r_2512
- R5: value 20k -> 10k; footprint pin_strip_3x2 -> R_Var
- R6: value 10k -> 120E; footprint rc03_vert -> r_0805
- R7: value 1k -> 15k; footprint rc03_vert -> r_0805
- U6: footprint DIP-8__300_ELL -> SO8E
Changed lines of the file:
@@
-EESchema Schematic File Version 2  date 7/19/2012 1:50:01 PM
+EESchema Schematic File Version 2  date 7/20/2012 2:32:56 PM
 LIBS:stfu
 LIBS:power
@@
 Sheet 2 3
 Title ""
-Date "19 jul 2012"
+Date "20 jul 2012"
 Rev ""
 Comp ""
@@
 F 0 "R43" V 8080 2650 50  0000 C CNN
 F 1 "220E" V 8000 2650 50  0000 C CNN
-F 2 "rc03_vert" H 8000 2650 60  0001 C CNN
+F 2 "r_0805" H 8000 2650 60  0001 C CNN
 	1    8000 2650
 	-1   0    0    1
@@
 F 0 "R42" V 7730 2650 50  0000 C CNN
 F 1 "47E" V 7650 2650 50  0000 C CNN
-F 2 "rc03_vert" H 7650 2650 60  0001 C CNN
+F 2 "r_2512" H 7650 2650 60  0001 C CNN
 	1    7650 2650
 	-1   0    0    1
@@
 F 0 "C9" H 4850 4500 50  0000 L CNN
 F 1 "1n" H 4850 4300 50  0000 L CNN
-F 2 "cnp_3mm_disc" H 4800 4400 60  0001 C CNN
+F 2 "c_0805" H 4800 4400 60  0001 C CNN
 	1    4800 4400
 	1    0    0    -1
@@
 F 0 "C10" H 5200 4500 50  0000 L CNN
 F 1 "47n" H 5200 4300 50  0000 L CNN
-F 2 "cnp_3mm_disc" H 5150 4400 60  0001 C CNN
+F 2 "c_0805" H 5150 4400 60  0001 C CNN
 	1    5150 4400
 	1    0    0    -1
@@
 F 0 "C6" H 4150 3850 50  0000 L CNN
 F 1 "100n" H 4150 3650 50  0000 L CNN
-F 2 "CP_5x11mm" H 4100 3750 60  0001 C CNN
+F 2 "c_0805" H 4100 3750 60  0001 C CNN
 	1    4100 3750
 	1    0    0    -1
@@
 P 4800 2650
 F 0 "R5" H 4900 2550 50  0000 C CNN
-F 1 "20k" V 4700 2650 50  0000 C CNN
-F 2 "pin_strip_3x2" H 4800 2650 60  0001 C CNN
+F 1 "10k" V 4700 2650 50  0000 C CNN
+F 2 "R_Var" H 4800 2650 60  0001 C CNN
 	1    4800 2650
 	1    0    0    -1
@@
 P 4800 3850
 F 0 "R7" H 4900 3950 50  0000 C CNN
-F 1 "1k" V 4800 3850 50  0000 C CNN
-F 2 "rc03_vert" H 4800 3850 60  0001 C CNN
+F 1 "15k" V 4800 3850 50  0000 C CNN
+F 2 "r_0805" H 4800 3850 60  0001 C CNN
 	1    4800 3850
 	1    0    0    -1
@@
 P 4800 3250
 F 0 "R6" H 4900 3350 50  0000 C CNN
-F 1 "10k" V 4800 3250 50  0000 C CNN
-F 2 "rc03_vert" H 4800 3250 60  0001 C CNN
+F 1 "120E" V 4800 3250 50  0000 C CNN
+F 2 "r_0805" H 4800 3250 60  0001 C CNN
 	1    4800 3250
 	1    0    0    -1
@@
 F 0 "R41" V 7080 3700 50  0000 C CNN
 F 1 "120E" V 7000 3700 50  0000 C CNN
-F 2 "rc03_vert" H 7000 3700 60  0001 C CNN
+F 2 "r_0805" H 7000 3700 60  0001 C CNN
 	1    7000 3700
 	0    -1   -1   0
@@
 F 0 "U6" H 6525 4250 60  0000 C CNN
 F 1 "NE555" H 6600 4150 60  0000 C CNN
-F 2 "DIP-8__300_ELL" H 6150 3800 60  0001 C CNN
+F 2 "SO8E" H 6150 3800 60  0001 C CNN
 	1    6150 3800
 	1    0    0    -1
